Commit message: T&W: transmission tower and grass in world. TODO: fix two missing lines in transmission tower and add more towers

File: models/rotors_description/urdf/iris_base.xacro (robot description, xacro)
@@ -96,4 +96,40 @@
   </xacro:mavlink_interface_macro>
   </xacro:if>
+  <xacro:camera_macro
+    namespace="${namespace}"
+    parent_link="base_link"
+    camera_suffix="left"
+    frame_rate="30.0"
+    horizontal_fov="1.3962634"
+    image_width="320"
+    image_height="240"
+    image_format="R8G8B8"
+    min_distance="0.02"
+    max_distance="100"
+    noise_mean="0.0"
+    noise_stddev="0.007"
+    enable_visual="1"
+    >
+    <box size="0.05 0.05 0.025" />
+    <origin xyz="0 0.07 -0.07" rpy="0 1.57079 0"/>
+  </xacro:camera_macro>
+    <xacro:camera_macro
+    namespace="${namespace}"
+    parent_link="base_link"
+    camera_suffix="right"
+    frame_rate="30.0"
+    horizontal_fov="1.3962634"
+    image_width="320"
+    image_height="240"
+    image_format="R8G8B8"
+    min_distance="0.02"
+    max_distance="100"
+    noise_mean="0.0"
+    noise_stddev="0.007"
+    enable_visual="1"
+    >
+    <box size="0.05 0.05 0.025" />
+    <origin xyz="0 -0.07 -0.07" rpy="0 1.57079 0"/>
+    </xacro:camera_macro>
   <!-- Mount an ADIS16448 IMU. -->
   <xacro:imu_plugin_macro

Commit message: T&W: PID adjusted

File: models/rotors_description/urdf/iris_base.xacro (robot description, xacro)
@@ -112,5 +112,5 @@
     >
     <box size="0.05 0.05 0.025" />
-    <origin xyz="0 0.07 -0.07" rpy="0 1.57079 0"/>
+    <origin xyz="0 0.095 -0.09" rpy="0 1.57079 0"/>
   </xacro:camera_macro>
     <xacro:camera_macro
@@ -130,5 +130,5 @@
     >
     <box size="0.05 0.05 0.025" />
-    <origin xyz="0 -0.07 -0.07" rpy="0 1.57079 0"/>
+    <origin xyz="0 -0.095 -0.09" rpy="0 1.57079 0"/>
     </xacro:camera_macro>
   <!-- Mount an ADIS16448 IMU. -->

File: models/rotors_description/urdf/multirotor_base.xacro (robot description, xacro)
@@ -123,9 +123,8 @@
         <motorSpeedPubTopic>/motor_speed/${motor_number}</motorSpeedPubTopic>
         <rotorVelocitySlowdownSim>${rotor_velocity_slowdown_sim}</rotorVelocitySlowdownSim>
-        <!--
         <gazebo_joint_control_pid>
           <p>0.1</p>
-          <i>0</i>
-          <d>0</d>
+          <i>0.02</i>
+          <d>0.001</d>
           <iMax>0</iMax>
           <iMin>0</iMin>
@@ -133,5 +132,4 @@
           <cmdMin>-3</cmdMin>
         </gazebo_joint_control_pid>
-      -->
       </plugin>
     </gazebo>
