Commit message: T&W: 3D lines with stereo vision

File: models/rotors_description/urdf/component_snippets.xacro (robot description, xacro)
@@ -62,5 +62,5 @@
       <xacro:insert_block name="origin" />
       <parent link="${parent_link}" />
-      <child link="${namespace}/camera_${camera_suffix}_link" />
+      <child link="/camera_${camera_suffix}_link" />
     </joint>
     <gazebo reference="${namespace}/camera_${camera_suffix}_link">
@@ -95,10 +95,10 @@
           <cameraInfoTopicName>camera_info</cameraInfoTopicName>
           <frameName>camera_${camera_suffix}_link</frameName>
-          <hackBaseline>0.0</hackBaseline>
+          <hackBaseline>0.19</hackBaseline>
           <distortionK1>0.0</distortionK1>
-          <distortionK2>0.0</distortionK2>
-          <distortionK3>0.0</distortionK3>
-          <distortionT1>0.0</distortionT1>
-          <distortionT2>0.0</distortionT2>
+          <distortionK2>0.272060548765299</distortionK2>
+          <distortionK3>-0.4510090027068866</distortionK3>
+          <distortionT1>0.001047801344634938</distortionT1>
+          <distortionT2>0.003251669895195926</distortionT2>
         </plugin>
       </sensor>

File: models/rotors_description/urdf/iris_base.xacro (robot description, xacro)
@@ -101,10 +101,10 @@
     camera_suffix="left"
     frame_rate="30.0"
-    horizontal_fov="1.3962634"
-    image_width="320"
-    image_height="240"
+    horizontal_fov="1.13446"
+    image_width="640"
+    image_height="480"
     image_format="R8G8B8"
     min_distance="0.02"
-    max_distance="100"
+    max_distance="50"
     noise_mean="0.0"
     noise_stddev="0.007"
@@ -119,10 +119,10 @@
     camera_suffix="right"
     frame_rate="30.0"
-    horizontal_fov="1.3962634"
-    image_width="320"
-    image_height="240"
+    horizontal_fov="1.13446"
+    image_width="640"
+    image_height="480"
     image_format="R8G8B8"
     min_distance="0.02"
-    max_distance="100"
+    max_distance="50"
     noise_mean="0.0"
     noise_stddev="0.007"
